File: NuttyHardware/esp32-s3.kicad_sch (KiCad schematic)
At the start: 44 parts, among them J9 USB Type-C Port, Q10 AO3401A, Q11 AO3400A, Q12 AO3401A, Q5 MMBT3904, Q8 MMBT3904, Q9 FDC6333C, SW11 BTN_RST, SW12 BTN_IO0, U10 CH334R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

Commit message: [HARDWARE] NuttyBadge Rev. C (May-2026)
Parts:
- C49, C51: value 15p -> NC
